File: temp0_schematic/temp0_schematic.sch (KiCad schematic (older format))
At the start: 18 parts, among them J1 MODE1_EXT, U1 Pro_Trinket_5V, U2 ESP-01, U3 oled_I2C_ssd1306, U4 hdc1080, U5 3.3V_REG, U6 ftdi_header

Commit message: Schematic and PCB revision 2.
Parts:
- removed ESP_PRG1, ESP_RST1: SW_Push, Button_Switch_SMD:SW_Push_1P1T_NO_6x6mm_H9.5mm, symbol Switch:SW_Push
- removed R2: 10k, Resistor_SMD:R_1206_3216Metric_Pad1.42x1.75mm_HandSolder, symbol Device:R
- removed U6: ftdi_header, Connector_PinHeader_2.54mm:PinHeader_1x06_P2.54mm_Horizontal, symbol temp0_parts:ftdi_header
Connections:
- net 3.3V: now also U2.6 (RST)
- no-connect marks 18 -> 17
Other:
- note added: "2"
- note added: "20200418"
- note added: "Changes from Rev: 1\n- Removed ftdi header for programming ESP8266.\n- Removed ESP8266 program button\n- Removed ESP8266 reset button"
- note added: "ESP8266 Module (ESP-01)"
- note removed: "1"
- note removed: "20200404"
- note removed: "ESP8266 Module (ESP-01)\nIncluding Serial Header for Programming"
- note removed: "Note: FTDI Header will only work\nfor serial comms to ESP-01.\nI.e. Tx/Rx are reversed as \nconnected to Pro Trinket"
- moved on the sheet: R3, R4
Changed lines of the file:
@@
-$EndComp
-$Comp
-L Switch:SW_Push ESP_RST1
-U 1 1 5E80A160
-P 3800 4950
-F 0 "ESP_RST1" H 3800 4900 50  0000 C CNN
-F 1 "SW_Push" H 3800 5150 50  0000 C CNN
-F 2 "Button_Switch_SMD:SW_Push_1P1T_NO_6x6mm_H9.5mm" H 3800 5150 50  0001 C CNN
-F 3 "~" H 3800 5150 50  0001 C CNN
-	1    3800 4950
-	1    0    0    -1
-$EndComp
-$Comp
-L Switch:SW_Push ESP_PRG1
-U 1 1 5E80A490
-P 2150 4950
-F 0 "ESP_PRG1" H 2150 4900 50  0000 C CNN
-F 1 "SW_Push" H 2150 5144 50  0000 C CNN
-F 2 "Button_Switch_SMD:SW_Push_1P1T_NO_6x6mm_H9.5mm" H 2150 5150 50  0001 C CNN
-F 3 "~" H 2150 5150 50  0001 C CNN
-	1    2150 4950
-	1    0    0    -1
 $EndComp
 $Comp
@@
 Text GLabel 6700 2700 2    50   Input ~ 0
 3.3V
-Text GLabel 3450 4550 2    50   Input ~ 0
+Text GLabel 3350 4850 2    50   Input ~ 0
 3.3V
 $Comp
@@
 	1    0    0    -1
 $EndComp
-$Comp
-L power:GND #PWR0102
-U 1 1 5E825495
-P 4050 5000
-F 0 "#PWR0102" H 4050 4750 50  0001 C CNN
-F 1 "GND" H 4055 4827 50  0000 C CNN
-F 2 "" H 4050 5000 50  0001 C CNN
-F 3 "" H 4050 5000 50  0001 C CNN
-	1    4050 5000
-	1    0    0    -1
-$EndComp
-$Comp
-L Device:R R2
-U 1 1 5E817911
-P 3400 4750
-F 0 "R2" H 3470 4796 50  0000 L CNN
-F 1 "10k" H 3470 4705 50  0000 L CNN
-F 2 "Resistor_SMD:R_1206_3216Metric_Pad1.42x1.75mm_HandSolder" V 3330 4750 50  0001 C CNN
-F 3 "~" H 3400 4750 50  0001 C CNN
-	1    3400 4750
-	1    0    0    -1
-$EndComp
-$Comp
-L power:GND #PWR0103
-U 1 1 5E82DB9D
-P 1900 5200
-F 0 "#PWR0103" H 1900 4950 50  0001 C CNN
-F 1 "GND" H 1905 5027 50  0000 C CNN
-F 2 "" H 1900 5200 50  0001 C CNN
-F 3 "" H 1900 5200 50  0001 C CNN
-	1    1900 5200
-	1    0    0    -1
-$EndComp
 Text GLabel 2750 2350 0    50   Input ~ 0
 U1_TX
-Text GLabel 1800 4250 2    50   Input ~ 0
+Text GLabel 2200 4350 2    50   Input ~ 0
 U1_TX
-Text GLabel 3350 5150 2    50   Input ~ 0
+Text GLabel 3300 5150 2    50   Input ~ 0
 U1_RX
-Wire Wire Line
-	3250 5150 3350 5150
 NoConn ~ 2400 5050
 $Comp
 L Device:R R3
 U 1 1 5E837B90
-P 1750 4850
-F 0 "R3" H 1820 4896 50  0000 L CNN
-F 1 "10k" H 1820 4805 50  0000 L CNN
-F 2 "Resistor_SMD:R_1206_3216Metric_Pad1.42x1.75mm_HandSolder" V 1680 4850 50  0001 C CNN
-F 3 "~" H 1750 4850 50  0001 C CNN
-	1    1750 4850
+P 2150 4950
+F 0 "R3" H 2220 4996 50  0000 L CNN
+F 1 "10k" H 2220 4905 50  0000 L CNN
+F 2 "Resistor_SMD:R_1206_3216Metric_Pad1.42x1.75mm_HandSolder" V 2080 4950 50  0001 C CNN
+F 3 "~" H 2150 4950 50  0001 C CNN
+	1    2150 4950
 	1    0    0    -1
 $EndComp
@@
 L Device:R R4
 U 1 1 5E8383EE
-P 1750 4450
-F 0 "R4" H 1820 4496 50  0000 L CNN
-F 1 "22k" H 1820 4405 50  0000 L CNN
-F 2 "Resistor_SMD:R_1206_3216Metric_Pad1.42x1.75mm_HandSolder" V 1680 4450 50  0001 C CNN
-F 3 "~" H 1750 4450 50  0001 C CNN
-	1    1750 4450
+P 2150 4550
+F 0 "R4" H 2220 4596 50  0000 L CNN
+F 1 "22k" H 2220 4505 50  0000 L CNN
+F 2 "Resistor_SMD:R_1206_3216Metric_Pad1.42x1.75mm_HandSolder" V 2080 4550 50  0001 C CNN
+F 3 "~" H 2150 4550 50  0001 C CNN
+	1    2150 4550
 	1    0    0    -1
 $EndComp
@@
 	0    -1   -1   0
 $EndComp
-Text GLabel 2500 5950 3    50   Input ~ 0
-U1_RX
-Text GLabel 2400 5950 3    50   Input ~ 0
-U1_TX
-Text GLabel 2300 5950 3    50   Input ~ 0
-3.3V
-$Comp
-L power:GND #PWR0107
-U 1 1 5E81FDC4
-P 2100 5950
-F 0 "#PWR0107" H 2100 5700 50  0001 C CNN
-F 1 "GND" H 2105 5777 50  0000 C CNN
-F 2 "" H 2100 5950 50  0001 C CNN
-F 3 "" H 2100 5950 50  0001 C CNN
-	1    2100 5950
-	1    0    0    -1
-$EndComp
-NoConn ~ 2600 5900
-NoConn ~ 2200 5900
-$Comp
-L temp0_parts:ftdi_header U6
-U 1 1 5E82DE8D
-P 2350 5650
-F 0 "U6" H 2300 5750 50  0000 L CNN
-F 1 "ftdi_header" H 2150 5850 50  0000 L CNN
-F 2 "Connector_PinHeader_2.54mm:PinHeader_1x06_P2.54mm_Horizontal" H 2350 5550 50  0001 C CNN
-F 3 "" H 2350 5550 50  0001 C CNN
-	1    2350 5650
-	1    0    0    -1
-$EndComp
 Wire Wire Line
 	2400 4850 2350 4850
-Wire Wire Line
-	2350 4850 2350 4650
-Wire Wire Line
-	2400 4950 2350 4950
-Wire Wire Line
-	1950 4950 1900 4950
-Wire Wire Line
-	1900 4950 1900 5150
-Connection ~ 1900 5150
-Wire Wire Line
-	1900 5150 2400 5150
-Wire Wire Line
-	1900 5200 1900 5150
-Wire Wire Line
-	1750 5000 1750 5150
-Wire Wire Line
-	1750 5150 1900 5150
-Wire Wire Line
-	1750 4700 1750 4650
-Wire Wire Line
-	2350 4650 1750 4650
-Connection ~ 1750 4650
-Wire Wire Line
-	1750 4650 1750 4600
-Wire Wire Line
-	1800 4250 1750 4250
-Wire Wire Line
-	1750 4250 1750 4300
-Wire Wire Line
-	2100 5950 2100 5900
-Wire Wire Line
-	2300 5900 2300 5950
-Wire Wire Line
-	2400 5950 2400 5900
-Wire Wire Line
-	2500 5900 2500 5950
 Wire Wire Line
 	2750 2350 2800 2350
@@
 Wire Notes Line
 	4400 1250 4400 3000
-Text Notes 2800 5900 0    50   ~ 0
-Note: FTDI Header will only work\nfor serial comms to ESP-01.\nI.e. Tx/Rx are reversed as \nconnected to Pro Trinket
 Text Notes 3050 2950 0    50   ~ 0
 Pro Trinket Module (Atemga328P)
-Text Notes 2550 4350 0    50   ~ 0
-ESP8266 Module (ESP-01)\nIncluding Serial Header for Programming
+Text Notes 3500 4550 2    50   ~ 0
+ESP8266 Module (ESP-01)
 Text Notes 5550 3600 0    50   ~ 0
 3.3V Power Regulator\nInput: 5V from USB (via Pro Trinket)\nOutput 3.3V to  ESP8266 and HDC1080
@@
 temp0 schematic
 Text Notes 8150 7650 0    79   ~ 0
-20200404
+20200418
 Text Notes 10550 7650 0    79   ~ 0
-1
+2
 Wire Notes Line
 	8200 3600 8200 2500
@@
 Wire Notes Line
 	9550 3600 8200 3600
-Wire Notes Line
-	1600 4150 1600 6300
 Wire Wire Line
 	2100 2550 2050 2550
@@
 Wire Wire Line
 	1550 2350 1550 2700
+NoConn ~ 2400 4950
+$Comp
+L power:GND #PWR0103
+U 1 1 5E82DB9D
+P 2150 5200
+F 0 "#PWR0103" H 2150 4950 50  0001 C CNN
+F 1 "GND" H 2155 5027 50  0000 C CNN
+F 2 "" H 2150 5200 50  0001 C CNN
+F 3 "" H 2150 5200 50  0001 C CNN
+	1    2150 5200
+	1    0    0    -1
+$EndComp
+Wire Wire Line
+	2400 5150 2150 5150
+Wire Wire Line
+	2150 5200 2150 5150
 Wire Wire Line
 	3250 5050 3300 5050
 Wire Wire Line
-	3300 5050 3300 4850
-Wire Wire Line
-	3300 4850 3250 4850
-Wire Wire Line
-	3250 4950 3400 4950
-Wire Wire Line
-	3450 4550 3400 4550
-Wire Wire Line
-	3300 4550 3300 4850
+	3300 5050 3300 4950
+Wire Wire Line
+	3300 4850 3350 4850
+Wire Wire Line
+	3250 4950 3300 4950
+Connection ~ 3300 4950
+Wire Wire Line
+	3300 4950 3300 4850
+Wire Wire Line
+	3250 4850 3300 4850
 Connection ~ 3300 4850
-Wire Wire Line
-	3400 4600 3400 4550
-Connection ~ 3400 4550
-Wire Wire Line
-	3400 4550 3300 4550
-Wire Wire Line
-	3400 4900 3400 4950
-Wire Wire Line
-	3600 4950 3400 4950
-Connection ~ 3400 4950
-Wire Wire Line
-	4050 5000 4050 4950
-Wire Wire Line
-	4050 4950 4000 4950
-Wire Notes Line
-	1600 4150 4150 4150
-Wire Notes Line
-	4150 4150 4150 6300
-Wire Notes Line
-	4150 6300 1600 6300
+Text Notes 7000 7000 0    50   ~ 0
+Changes from Rev: 1\n- Removed ftdi header for programming ESP8266.\n- Removed ESP8266 program button\n- Removed ESP8266 reset button
+Wire Wire Line
+	2150 5150 2150 5100
+Connection ~ 2150 5150
+Wire Wire Line
+	2350 4850 2350 4750
+Wire Wire Line
+	2350 4750 2150 4750
+Wire Wire Line
+	2150 4750 2150 4800
+Wire Wire Line
+	2150 4700 2150 4750
+Connection ~ 2150 4750
+Wire Wire Line
+	2200 4350 2150 4350
+Wire Wire Line
+	2150 4350 2150 4400
+Wire Wire Line
+	3250 5150 3300 5150
+Wire Notes Line
+	2050 4250 2050 5450
+Wire Notes Line
+	2050 5450 3650 5450
+Wire Notes Line
+	3650 5450 3650 4250
+Wire Notes Line
+	3650 4250 2050 4250
 $EndSCHEMATC
